File: left_110key/left_110key.kicad_pcb (KiCad board)
At the start: 2 copper layers, 428.1 x 121 mm, 358 parts, among them J1 Conn_01x04_Male, J10 Conn_01x04_Male, J100 Conn_01x04_Male, J101 Conn_01x04_Male, J102 Conn_01x04_Male, J103 Conn_01x04_Male, J104 Conn_01x04_Male, J105 Conn_01x04_Male, J106 Conn_01x04_Male, J107 Conn_01x04_Male, J108 Conn_01x04_Male, J109 Conn_01x04_Male, J11 Conn_01x04_Male, J110 Conn_01x04_Male, J12 Conn_01x04_Male, J13 Conn_01x04_Male, J14 Conn_01x04_Male, J15 Conn_01x04_Male, J16 Conn_01x04_Male, J17 Conn_01x04_Male, J18 Conn_01x04_Male, J19 Conn_01x04_Male, J2 Conn_01x04_Male, J20 Conn_01x04_Male, J21 Conn_01x04_Male, J22 Conn_01x04_Male, J23 Conn_01x04_Male, J24 Conn_01x04_Male, J25 Conn_01x04_Male, J26 Conn_01x04_Male, J27 Conn_01x04_Male, J28 Conn_01x04_Male, J29 Conn_01x04_Male, J3 Conn_01x04_Male, J30 Conn_01x04_Male, J31 Conn_01x04_Male, J32 Conn_01x04_Male, J33 Conn_01x04_Male, J34 Conn_01x04_Male, J35 Conn_01x04_Male, J36 Conn_01x04_Male, J37 Conn_01x04_Male, J38 Conn_01x04_Male, J39 Conn_01x04_Male, J4 Conn_01x04_Male, J40 Conn_01x04_Male, J41 Conn_01x04_Male, J42 Conn_01x04_Male, J43 Conn_01x04_Male, J44 Conn_01x04_Male, J45 Conn_01x04_Male, J46 Conn_01x04_Male, J47 Conn_01x04_Male, J48 Conn_01x04_Male, J49 Conn_01x04_Male, J5 Conn_01x04_Male, J50 Conn_01x04_Male, J51 Conn_01x04_Male, J52 Conn_01x04_Male, J53 Conn_01x04_Male, J54 Conn_01x04_Male, J55 Conn_01x04_Male, J56 Conn_01x04_Male, J57 Conn_01x04_Male, J58 Conn_01x04_Male, J59 Conn_01x04_Male, J6 Conn_01x04_Male, J60 Conn_01x04_Male, J61 Conn_01x04_Male, J62 Conn_01x04_Male, J63 Conn_01x04_Male, J64 Conn_01x04_Male, J65 Conn_01x04_Male, J66 Conn_01x04_Male, J67 Conn_01x04_Male, J68 Conn_01x04_Male, J69 Conn_01x04_Male, J7 Conn_01x04_Male, J70 Conn_01x04_Male, J71 Conn_01x04_Male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

Commit message: Add files via upload
Parts:
- moved REF** 5.81 mm to (177.8, 193.7)
- moved REF** 1.56 mm to (370.0, 164.3)
- moved REF** 0.96 mm to (370.7, 102.4)

Commit message: Add files via upload
Routing:
- net Net-(R113-Pad1): track 26.6 -> 47.2 mm
- net Net-(D113-Pad2): track 29.4 -> 28.8 mm
