File: mouse8onethreev2/mouse8.kicad_pcb (KiCad board)
At the start: 2 copper layers, 94 x 44.5 mm, 62 parts, among them J1 Conn_01x05_Female, J2 Conn_01x05_Female, J3 Conn_01x01, J4 Conn_01x01, J6 Conn_01x01, J7 Conn_01x02_Female, J8 Conn_01x02_Female, J9 Conn_01x02_Female, SW1 SW_SPST, SW2 SW_SPST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

Commit message: Add files via upload
Parts:
- removed C13: 0.1uF, Capacitor_SMD:C_0805_2012Metric_Pad1.15x1.40mm_HandSolder
- C12: value 10uF -> 1uF
- U4: value TPS73601DBV -> RT9179GB
- moved C12 9.65 mm to (79.3, -48.5)
- moved SW1 2.26 mm to (129.7, -67.6)
Routing:
- net Net-(C12-Pad1): track 108.9 -> 97.3 mm
- net Net-(R20-Pad1): track 7.96 -> 6.07 mm
