File: mouse8onethreev2/mouse8.sch (KiCad schematic (older format))
At the start: 62 parts, among them J1 Conn_01x05_Female, J2 Conn_01x05_Female, J3 Conn_01x01, J4 Conn_01x01, J6 Conn_01x01, J7 Conn_01x02_Female, J8 Conn_01x02_Female, J9 Conn_01x02_Female, SW1 SW_SPST, SW2 SW_SPST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

Commit message: Add files via upload
Parts:
- removed C13: 0.1uF, Capacitor_SMD:C_0805_2012Metric_Pad1.15x1.40mm_HandSolder, symbol Device:C
- C12: value 10uF -> 1uF; Field4 C15850 -> C28323
- U4: value TPS73601DBV -> RT9179GB; Field4 C59200 -> C130831
Changed lines of the file:
@@
 P 5200 2550
 F 0 "C12" H 5025 2625 50  0000 L CNN
-F 1 "10uF" H 5000 2475 50  0000 L CNN
+F 1 "1uF" H 5000 2475 50  0000 L CNN
 F 2 "Capacitor_SMD:C_0805_2012Metric_Pad1.15x1.40mm_HandSolder" H 5238 2400 50  0001 C CNN
 F 3 "~" H 5200 2550 50  0001 C CNN
-F 4 "C15850" H 5200 2550 50  0001 C CNN "Field4"
+F 4 "C28323" H 5200 2550 50  0001 C CNN "Field4"
 	1    5200 2550
 	1    0    0    -1
@@
 P 4400 1850
 F 0 "U4" H 4400 2217 50  0000 C CNN
-F 1 "TPS73601DBV" H 4400 2126 50  0000 C CNN
+F 1 "RT9179GB" H 4400 2126 50  0000 C CNN
 F 2 "Package_TO_SOT_SMD:SOT-23-5" H 4400 2175 50  0001 C CIN
 F 3 "http://www.ti.com/lit/ds/symlink/tps736.pdf" H 4400 1800 50  0001 C CNN
-F 4 "C59200" H 4400 1850 50  0001 C CNN "Field4"
+F 4 "C130831" H 4400 1850 50  0001 C CNN "Field4"
 	1    4400 1850
 	1    0    0    -1
@@
 Wire Wire Line
 	4800 1625 3850 1625
-$Comp
-L Device:C C13
-U 1 1 5DE47F21
-P 4900 1775
-F 0 "C13" H 4900 1850 50  0000 L CNN
-F 1 "0.1uF" H 4825 2000 50  0000 L CNN
-F 2 "Capacitor_SMD:C_0805_2012Metric_Pad1.15x1.40mm_HandSolder" H 4938 1625 50  0001 C CNN
-F 3 "~" H 4900 1775 50  0001 C CNN
-F 4 "C49678" H 4900 1775 50  0001 C CNN "Field4"
-	1    4900 1775
-	1    0    0    -1
-$EndComp
-Connection ~ 4900 1625
-Wire Wire Line
-	4900 1625 4800 1625
-Wire Wire Line
-	4900 1925 4900 2050
 Wire Wire Line
 	5350 3150 5350 1450
@@
 Wire Wire Line
 	5200 1625 5200 2050
-Connection ~ 4900 2050
 Connection ~ 5200 2050
 Wire Wire Line
 	5200 2050 5200 2400
-Wire Wire Line
-	4900 1625 5200 1625
 Connection ~ 4250 2900
 Wire Wire Line
@@
 Wire Wire Line
 	3275 2400 3150 2400
+Wire Wire Line
+	4800 1625 5200 1625
 $EndSCHEMATC
